File: PCB/HKI-KTS-1.kicad_sch (KiCad schematic)
At the start: 59 parts

Commit message: pcb changes
Parts:
- removed C4001, C4004, C4007: 10uF, PCM_JLCPCB:C_0402, symbol PCM_JLCPCB-Capacitors:0402,10uF
- removed C4002, C4003, C4005, C4006, C4008, C4009: 220nF, PCM_JLCPCB:C_0402, symbol PCM_JLCPCB-Capacitors:0402,220nF
- added C43, C44, C45, C46, C47, C48, C49, C50, C51: 1uF, PCM_JLCPCB:C_0402, symbol PCM_JLCPCB-Capacitors:0402,1uF
- renumbered D4001 to D143, D4002 to D144, D4003 to D145, D4004 to D146, D4005 to D147, D4006 to D148, D4007 to D149, D4008 to D150, D4009 to D151, D4010 to D152, D4011 to D153, D4012 to D154, D4013 to D155, D4014 to D156, D4015 to D157, D4016 to D158, D4017 to D159, D4018 to D160, D4019 to D161, D4020 to D162, D4021 to D163, D4022 to D164, D4023 to D165, D4024 to D166, D4025 to D167, D4026 to D168, D4027 to D169, D4028 to D170, D4029 to D171, D4030 to D172, D4031 to D173, D4032 to D174, D4033 to D175, D4034 to D176, D4035 to D177, D4036 to D178, D4037 to D179, D4038 to D180, D4039 to D181, D4040 to D182, D4041 to D183, D4042 to D184, D4043 to D185, D4044 to D186, D4045 to D187, D4046 to D188, D4047 to D189, D4048 to D190, D4049 to D191, D4050 to D192
Connections:
- net +5V: now also C43.1, C44.1, C45.1, C46.1, C47.1, C48.1, C49.1, C50.1, C51.1
- net GND: now also C43.2, C44.2, C45.2, C46.2, C47.2, C48.2, C49.2, C50.2, C51.2
