File: PCB/HKI-KTS-2.kicad_sch (KiCad schematic)
At the start: 64 parts

Commit message: pcb changes
Parts:
- removed C5001, C5004, C5007: 10uF, PCM_JLCPCB:C_0402, symbol PCM_JLCPCB-Capacitors:0402,10uF
- removed C5002, C5003, C5005, C5006, C5008, C5009: 220nF, PCM_JLCPCB:C_0402, symbol PCM_JLCPCB-Capacitors:0402,220nF
- added C52, C53, C54: 1uF, PCM_JLCPCB:C_0402, symbol PCM_JLCPCB-Capacitors:0402,1uF
- renumbered D5001 to D193, D5002 to D194, D5003 to D195, D5004 to D196, D5005 to D197, D5006 to D198, D5007 to D199, D5008 to D200, D5009 to D201, D5010 to D202, D5011 to D203, D5012 to D204, D5013 to D205, D5014 to D206, D5015 to D207, D5016 to D208, D5017 to D209, D5018 to D210, D5019 to D211, D5020 to D212, D5021 to D213, D5022 to D214, D5023 to D215, D5024 to D216, D5025 to D217, D5026 to D218, D5027 to D219, D5028 to D220, D5029 to D221, D5030 to D222, D5031 to D223, D5032 to D224, D5033 to D225, D5034 to D226, D5035 to D227, D5036 to D228, D5037 to D229, D5038 to D230, D5039 to D231, D5040 to D232, D5041 to D233, D5042 to D234, D5043 to D235, D5044 to D236, D5045 to D237, D5046 to D238, D5047 to D239, D5048 to D240, D5050 to D241, D5051 to D242, D5052 to D243, D5053 to D244, D5054 to D245, D5055 to D246, D5056 to D247
Connections:
- net +5V: now also C52.1, C53.1, C54.1
- net GND: now also C52.2, C53.2, C54.2
