File: PCB/HKI-KTS-3.kicad_sch (KiCad schematic)
At the start: 55 parts

Commit message: pcb fixes
Parts:
- added D6013: WS2812B, PCM_JLCPCB:LED-SMD_4P-L1.6-W1.5_XL-1615RGBC-WS2812B, symbol PCM_JLCPCB-Extended:LED, WS2812B, 1615
Connections:
- net +5V: now also D6013.2 (VDD)
- net GND: now also D6013.1 (DOUT), D6013.3 (GND); no longer D6044.1 (DOUT)
- new net: D6013.4 (DIN), D6044.1 (DOUT)
Other:
- moved on the sheet: C6001, C6002, C6003, C6004, C6005, C6006

Commit message: pcb changes
Parts:
- removed C6001, C6004: 10uF, PCM_JLCPCB:C_0402, symbol PCM_JLCPCB-Capacitors:0402,10uF
- removed C6002, C6003, C6005, C6006: 220nF, PCM_JLCPCB:C_0402, symbol PCM_JLCPCB-Capacitors:0402,220nF
- added C55, C56, C57, C58, C59, C60: 1uF, PCM_JLCPCB:C_0402, symbol PCM_JLCPCB-Capacitors:0402,1uF
- renumbered D6001 to D248, D6002 to D249, D6003 to D250, D6004 to D251, D6005 to D252, D6006 to D253, D6007 to D254, D6008 to D255, D6009 to D256, D6010 to D257, D6011 to D258, D6012 to D259, D6045 to D260, D6024 to D261, D6046 to D262, D6047 to D263, D6048 to D264, D6049 to D265, D6050 to D266, D6014 to D267, D6015 to D268, D6016 to D269, D6017 to D270, D6018 to D271, D6019 to D272, D6020 to D273, D6021 to D274, D6022 to D275, D6023 to D276, D6025 to D277, D6026 to D278, D6027 to D279, D6028 to D280, D6029 to D281, D6030 to D282, D6031 to D283, D6032 to D284, D6033 to D285, D6034 to D286, D6035 to D287, D6036 to D288, D6037 to D289, D6038 to D290, D6039 to D291, D6040 to D292, D6041 to D293, D6042 to D294, D6043 to D295, D6044 to D296, D6013 to D297
Connections:
- net +5V: now also C55.1, C56.1, C57.1, C58.1, C59.1, C60.1
- net GND: now also C55.2, C56.2, C57.2, C58.2, C59.2, C60.2

Commit message: Simulator added
Parts:
- removed D280: WS2812B, PCM_JLCPCB:LED-SMD_4P-L1.6-W1.5_XL-1615RGBC-WS2812B, symbol PCM_JLCPCB-Extended:LED, WS2812B, 1615
Connections:
- net at D289.1 (DOUT): now also D281.4 (DIN)
