File: PCB/HPL-NOA-1.kicad_sch (KiCad schematic)
At the start: 74 parts

Commit message: pcb changes
Parts:
- removed C2001, C2004, C2007: 10uF, PCM_JLCPCB:C_0402, symbol PCM_JLCPCB-Capacitors:0402,10uF
- removed C2002, C2003, C2005, C2006, C2008, C2009: 220nF, PCM_JLCPCB:C_0402, symbol PCM_JLCPCB-Capacitors:0402,220nF
- added C25, C26, C27, C28, C29, C30, C31, C32, C33: 1uF, PCM_JLCPCB:C_0402, symbol PCM_JLCPCB-Capacitors:0402,1uF
- renumbered D2001 to D13, D2002 to D14, D2003 to D15, D2004 to D16, D2005 to D17, D2006 to D18, D2007 to D19, D2008 to D20, D2009 to D21, D2010 to D22, D2011 to D23, D2012 to D24, D2013 to D25, D2014 to D26, D2015 to D27, D2016 to D28, D2017 to D29, D2018 to D30, D2019 to D31, D2020 to D32, D2021 to D33, D2022 to D34, D2023 to D35, D2024 to D36, D2025 to D37, D2026 to D38, D2027 to D39, D2028 to D40, D2029 to D41, D2030 to D42, D2031 to D43, D2032 to D44, D2033 to D45, D2034 to D46, D2035 to D47, D2036 to D48, D2037 to D49, D2038 to D50, D2039 to D51, D2040 to D52, D2065 to D53, D2041 to D54, D2042 to D55, D2043 to D56, D2044 to D57, D2045 to D58, D2046 to D59, D2047 to D60, D2048 to D61, D2049 to D62, D2050 to D63, D2051 to D64, D2052 to D65, D2053 to D66, D2054 to D67, D2055 to D68, D2056 to D69, D2057 to D70, D2058 to D71, D2059 to D72, D2060 to D73, D2061 to D74, D2062 to D75, D2063 to D76, D2064 to D77
Connections:
- net +5V: now also C25.1, C26.1, C27.1, C28.1, C29.1, C30.1, C31.1, C32.1, C33.1
- net GND: now also C25.2, C26.2, C27.2, C28.2, C29.2, C30.2, C31.2, C32.2, C33.2

Commit message: Simulator added
Parts:
- removed D33, D51: WS2812B, PCM_JLCPCB:LED-SMD_4P-L1.6-W1.5_XL-1615RGBC-WS2812B, symbol PCM_JLCPCB-Extended:LED, WS2812B, 1615
Connections:
- net at D52.4 (DIN): now also D50.1 (DOUT)
- net at D32.1 (DOUT): now also D34.4 (DIN)
