File: PCB/HPL-NOA-2.kicad_sch (KiCad schematic)
At the start: 74 parts

Commit message: pcb changes
Parts:
- removed C3001, C3004, C3007: 10uF, PCM_JLCPCB:C_0402, symbol PCM_JLCPCB-Capacitors:0402,10uF
- removed C3002, C3003, C3005, C3006, C3008, C3009: 220nF, PCM_JLCPCB:C_0402, symbol PCM_JLCPCB-Capacitors:0402,220nF
- added C34, C35, C36, C37, C38, C39, C40, C41, C42: 1uF, PCM_JLCPCB:C_0402, symbol PCM_JLCPCB-Capacitors:0402,1uF
- renumbered D3023 to D100, D3024 to D101, D3025 to D102, D3026 to D103, D3027 to D104, D3028 to D105, D3029 to D106, D3030 to D107, D3031 to D108, D3032 to D109, D3033 to D110, D3034 to D111, D3035 to D112, D3036 to D113, D3037 to D114, D3038 to D115, D3039 to D116, D3040 to D117, D3041 to D118, D3042 to D119, D3043 to D120, D3044 to D121, D3045 to D122, D3046 to D123, D3047 to D124, D3048 to D125, D3049 to D126, D3050 to D127, D3051 to D128, D3052 to D129, D3053 to D130, D3054 to D131, D3055 to D132, D3056 to D133, D3057 to D134, D3058 to D135, D3059 to D136, D3060 to D137, D3061 to D138, D3062 to D139, D3063 to D140, D3064 to D141, D3065 to D142, D3001 to D78, D3002 to D79, D3003 to D80, D3004 to D81, D3005 to D82, D3006 to D83, D3007 to D84, D3008 to D85, D3009 to D86, D3010 to D87, D3011 to D88, D3012 to D89, D3013 to D90, D3014 to D91, D3015 to D92, D3016 to D93, D3017 to D94, D3018 to D95, D3019 to D96, D3020 to D97, D3021 to D98, D3022 to D99
Connections:
- net +5V: now also C34.1, C35.1, C36.1, C37.1, C38.1, C39.1, C40.1, C41.1, C42.1
- net GND: now also C34.2, C35.2, C36.2, C37.2, C38.2, C39.2, C40.2, C41.2, C42.2
