File: PCB/HPL-NOA-3.kicad_sch (KiCad schematic)
At the start: 10 parts

Commit message: pcb fixes
Parts:
- removed D7002: WS2812B, PCM_JLCPCB:LED-SMD_4P-L1.6-W1.5_XL-1615RGBC-WS2812B, symbol PCM_JLCPCB-Extended:LED, WS2812B, 1615
Connections:
- net at D7003.4 (DIN): now also D7007.1 (DOUT)

Commit message: pcb changes
Parts:
- removed C7001: 10uF, PCM_JLCPCB:C_0402, symbol PCM_JLCPCB-Capacitors:0402,10uF
- removed C7002, C7003: 220nF, PCM_JLCPCB:C_0402, symbol PCM_JLCPCB-Capacitors:0402,220nF
- renumbered D7001 to D298, D7003 to D299, D7004 to D300, D7005 to D301, D7006 to D302, D7007 to D303
