File: PCB/Helsinki-LED-Train-Map.kicad_pcb (KiCad board)
At the start: 2 copper layers, 249 x 71.5 mm, 424 parts, among them J1 Prog Connector, Q1 HL3415A, Q2 MMBT3904, U1 XC6206P332MR, U2 Connector, USB-TYPE-C-16P, U3 ESP32-C3FH4, U4 Connector, USB-TYPE-C-16P, U5 SN74LVC4245APWR, X1 40MHz, 15pF

Commit message: Simulator added
Parts:
- removed D280, D33, D51: WS2812B, PCM_JLCPCB:LED-SMD_4P-L1.6-W1.5_XL-1615RGBC-WS2812B
- moved C30 7.27 mm to (88.2, 80.5), turned to 90 degrees
- moved C29 6.48 mm to (87.2, 80.5), turned to 90 degrees
- moved C28 6.24 mm to (86.2, 80.5), turned to 90 degrees
- moved C31 4.86 mm to (69.8, 63.2)
- moved C33 4.86 mm to (69.8, 65.2)
- moved C32 4.86 mm to (69.8, 64.2)
- moved D50 3.49 mm to (69.9, 60.5)
- moved D34 3.23 mm to (112.1, 58.6)
- moved D35 3.23 mm to (110.1, 56.7)
- moved D36 3.23 mm to (107.3, 56.0)
- moved D37 3.23 mm to (104.5, 56.0)
- moved D38 3.23 mm to (101.7, 56.0)
- moved D39 3.23 mm to (98.9, 56.0)
- moved D40 3.23 mm to (96.1, 56.0)
- moved D41 3.23 mm to (93.3, 56.0)
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Connections:
- D281 pad 4: Net-(D280-DOUT) -> Net-(D281-DIN)
- D289 pad 1: Net-(D280-DIN) -> Net-(D281-DIN)
- D34 pad 4: Net-(D33-DOUT) -> Net-(D32-DOUT)
- D52 pad 4: Net-(D51-DOUT) -> Net-(D50-DOUT)
Routing:
- net +5V: track 1544.8 -> 1535.1 mm, vias 286 -> 281
- net GND: track 87.6 -> 95.3 mm, vias 264 -> 258
- net Net-(D281-DIN): track 0.00 -> 6.27 mm, vias 0 -> 2
- net Net-(D280-DOUT): track 4.25 -> 0.00 mm
- net Net-(D299-DIN): track 2.91 -> 5.71 mm, vias 0 -> 2
- net Net-(D50-DOUT): track 3.88 -> 1.33 mm, vias 2 -> 0
- net Net-(D32-DOUT): track 4.67 -> 2.13 mm, vias 2 -> 0
- net Net-(D51-DOUT): track 2.02 -> 0.00 mm
- net Net-(D280-DIN): track 1.96 -> 0.00 mm
- net Net-(D33-DOUT): track 1.92 -> 0.00 mm
- net /MAP_MODE_BUTTON: track 310.2 -> 312.1 mm
- net HKI-KTS-1: track 63.1 -> 64.9 mm
- net /D+: track 90.4 -> 92.3 mm
- net VBUS: track 341.3 -> 343.2 mm
- net /WIFI_LED: track 274.0 -> 275.8 mm
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Other:
- board text added: "HSL- ja VR-lähijunaliikenne"
- board text added: "Hanko-Pohjoinen"
- board text added: "Inkoo"
- board text added: "Siuntio"
- board text removed: "Hanko-pohjoinen"
- board text removed: "Helsingin seudun lähijunakartta"
