File: PCB/Helsinki-LED-Train-Map.kicad_sch (KiCad schematic)
At the start: 94 parts, among them J1001 Prog Connector, Q1001 HL3415A, Q1002 MMBT3904, U1001 XC6206P332MR, U1002 Connector, USB-TYPE-C-16P, U1003 ESP32-C3FH4, U1004 Connector, USB-TYPE-C-16P, U1005 SN74LVC4245APWR, X1001 40MHz, 15pF

Commit message: pcb changes
Parts:
- removed C1002, C1003, C1008, C1010, C1011, C1015, C1020, C1023, C1024: 100nF, PCM_JLCPCB:C_0402, symbol PCM_JLCPCB-Capacitors:0402,100nF
- removed C1004, C1006, C1007, C1014: 10uF, PCM_JLCPCB:C_0402, symbol PCM_JLCPCB-Capacitors:0402,10uF
- removed C1012: 10nF, PCM_JLCPCB:C_0402, symbol PCM_JLCPCB-Capacitors:0402,10nF
- removed C1017, C1018: C_Small, PCM_JLCPCB:C_0402, symbol Device:C_Small
- removed FB1001: ~, PCM_JLCPCB:FB_0603, symbol PCM_JLCPCB-Inductors:Ferrite,0603,(2)
- removed H1001, H1002, H1003: ~, PCM_JLCPCB:Hole_Tooling_JLCPCB, symbol PCM_JLCPCB-Manufacturing:Tooling Hole, PCM_JLCPCB, 1.152mm
- removed R1001: 15kΩ, PCM_JLCPCB:R_0402, symbol PCM_JLCPCB-Resistors:0402,15kΩ
- removed R1008, R1009, R1010, R1016: 0Ω, PCM_JLCPCB:R_0402, symbol PCM_JLCPCB-Resistors:0402,0Ω
- removed R1015: 1kΩ, PCM_JLCPCB:R_0402, symbol PCM_JLCPCB-Resistors:0402,1kΩ
- added C10, C11, C12, C14, C19, C2, C20, C3, C5, C6, C7, C8: 1uF, PCM_JLCPCB:C_0402, symbol PCM_JLCPCB-Capacitors:0402,1uF
- added R1: 10kΩ, PCM_JLCPCB:R_0402, symbol PCM_JLCPCB-Resistors:0402,10kΩ
- added R13: 510Ω, PCM_JLCPCB:R_0402, symbol PCM_JLCPCB-Resistors:0402,510Ω
- added S4: Tactile Button, 160gf, PCM_JLCPCB:SW-SMD_4P-L5.1-W5.1-P3.70-LS6.5-TL-2, symbol PCM_JLCPCB-Connectors_Buttons:Tactile Button, 160gf
- renumbered AE1001 to AE1, C1001 to C1, C1013 to C13, C1016 to C15, C1019 to C16, C1021 to C17, C1022 to C18, C1025 to C21, C1026 to C22, C1027 to C23, C1028 to C24, C1005 to C4, C1009 to C9, D1001 to D1, D1010 to D10, D1011 to D11, D1012 to D12, D1002 to D2, D1003 to D3, D1004 to D4, D1005 to D5, D1006 to D6, D1007 to D7, D1008 to D8, D1009 to D9, F1001 to F1, J1001 to J1, L1001 to L1, L1002 to L2, L1003 to L3, PN1001 to PN1, Q1001 to Q1, Q1002 to Q2, R1012 to R10, R1013 to R11, R1014 to R12, R1017 to R14, R1018 to R15, R1019 to R16, R1020 to R17, R1021 to R18, R1022 to R19, R1002 to R2, R1023 to R20, R1024 to R21, R1025 to R22, R1026 to R23, R1003 to R3, R1004 to R4, R1005 to R5, R1006 to R6, R1007 to R7, R1011 to R9, S1001 to S1, S1002 to S2, S1003 to S3, TP1001 to TP1, TP1002 to TP2, TP1003 to TP3, TP1004 to TP4, TP1005 to TP5, TP1006 to TP6, U1001 to U1, U1002 to U2, U1003 to U3, U1004 to U4, U1005 to U5, X1001 to X1
Connections:
- net MCU_D+ is gone; now on net D+: U3.26 (GPIO19/USB_D+)
- net MCU_D- is gone; now on net D-: U3.25 (GPIO18/USB_D-)
- net +3V3: now also C10.1, C11.1, C12.1, C14.1, C20.1, C3.1, C5.1, C6.1, C7.1, C8.1
- net GND: now also U5.2 (DIR), C10.2, C11.2, C12.2, C14.2, C19.2, C2.2, C20.2, C3.2, C5.2, C6.2, C7.2, C8.2, S4.3 (C), S4.4 (D)
- net LED_+5V_EN_Active_High: now also R13.2
- net Reset: now also U3.7 (CHIP_EN)
- net VBUS: now also C19.1, C2.1, R1.1
- net at C22.1, Q2.1 (B): now also R13.1
- net at D1.1, D2.2, D5.1: now also F1.1
- net MAP_MODE_BUTTON: now reaches R5.2, U3.14 (GPIO8)
- net MAP_MODE_BUTTON: now also S4.1 (A), S4.2 (B)
- net at D2.1: now also R1.2

Commit message: readme changes
Connections:
- net NAL-NIMT_MCU renamed HPL-NOA_MCU
- net STRAND-MNK_MCU renamed HKI-KTS_MCU
Changed lines of the file:
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@@
 	(title_block
 		(title "Helsinki Region Live Train Map")
-		(date "2025-06-28")
+		(date "2025-07-19")
 		(rev "1")
 		(comment 1 "©Chris Dirks & Unto Ahti")
@@
 		)
 	)
-	(label "NAL-NIMT_MCU"
+	(label "HPL-NOA_MCU"
 		(at 241.3 134.62 0)
 		(effects
@@
 		)
 	)
-	(label "STRAND-MNK_MCU"
+	(label "HKI-KTS_MCU"
 		(at 205.74 73.66 180)
 		(effects
@@
 		)
 	)
-	(label "STRAND-MNK_MCU"
+	(label "HKI-KTS_MCU"
 		(at 241.3 132.08 0)
 		(effects
@@
 		)
 	)
-	(label "NAL-NIMT_MCU"
+	(label "HPL-NOA_MCU"
 		(at 187.96 45.72 0)
 		(effects
